File: EDDIE/ServoControllerCircuit.brd (EAGLE design)
At the start: 58.8 x 65.7 mm, 31 parts, among them Q1 20MHz, T1 2N3904, X1 SIGNAL-PWR-GND, X2 SIGNAL-PWR-GND

Commit message: Removed TX circuitry and moved cost analysis
Since the TX functionality for the PIC was not tested, I decided to remove it. It is also the case that the cost analysis file for Jim, which is currently in progress, was moved to the Document repository.
Parts:
- removed MIDI_PIN_TX-2, MIDI_PIN_TX-4, MIDI_PIN_TX-5: (no value), wirepad:2,15/1,0
- removed R8, R9: 220, resistor:0207/12
Connections:
- removed net N$11: MIDI_PIN_TX-5.1, R8.1
- removed net N$12: MIDI_PIN_TX-4.1, R9.1
- removed net TX_PIN: PIC16F628A.8, R8.2
- net +5V: no longer R9.2
- net GND: no longer MIDI_PIN_TX-2.1
Routing:
- net TX_PIN: track 9.98 -> 0.00 mm
- net N$12: track 6.55 -> 0.00 mm
- net N$11: track 5.08 -> 0.00 mm
Changed lines of the file:
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@@
 <attribute name="VALUE" x="5.08" y="17.78" size="0.0254" layer="27"/>
-</element>
-<element name="MIDI_PIN_TX-2" library="wirepad" package="2,15/1,0" value="" x="8.13" y="5.7" smashed="yes" rot="R180">
-<attribute name="NAME" x="2.727" y="8.697" size="1.016" layer="25" ratio="10"/>
-<attribute name="VALUE" x="8.13" y="4.7" size="0.0254" layer="27" rot="R180"/>
-</element>
-<element name="MIDI_PIN_TX-4" library="wirepad" package="2,15/1,0" value="" x="13.02" y="5.78" smashed="yes" rot="R180">
-<attribute name="NAME" x="18.163" y="3.383" size="1.016" layer="25" ratio="10" rot="R180"/>
-<attribute name="VALUE" x="13.02" y="4.78" size="0.0254" layer="27" rot="R180"/>
-</element>
-<element name="MIDI_PIN_TX-5" library="wirepad" package="2,15/1,0" value="" x="13.13" y="14.32" smashed="yes" rot="R180">
-<attribute name="NAME" x="16.273" y="11.923" size="1.016" layer="25" ratio="10" rot="R180"/>
-<attribute name="VALUE" x="13.13" y="13.32" size="0.0254" layer="27" rot="R180"/>
 </element>
 <element name="PIC16F628A" library="ic-package" package="SOCKET-18" value="" x="39.45" y="30.02" rot="R270"/>
@@
 <element name="R7" library="resistor" package="0207/12" value="100" x="48.69" y="5.08" smashed="yes" rot="R180">
 <attribute name="NAME" x="51.865" y="3.683" size="1.27" layer="25" ratio="10" rot="R180"/>
-</element>
-<element name="R8" library="resistor" package="0207/12" value="220" x="24.48" y="14.4" smashed="yes">
-<attribute name="NAME" x="21.305" y="15.797" size="1.27" layer="25" ratio="10"/>
-</element>
-<element name="R9" library="resistor" package="0207/12" value="220" x="24.18" y="10.16" smashed="yes">
-<attribute name="NAME" x="21.005" y="11.557" size="1.27" layer="25" ratio="10"/>
 </element>
 <element name="T1" library="transistor" package="TO92" value="2N3904" x="36.99" y="5.08" smashed="yes">
@@
 <contactref element="LED1" pad="K"/>
 <contactref element="LED2" pad="K"/>
-<contactref element="R9" pad="2"/>
 <polygon width="0.254" layer="1" isolate="0.6096" orphans="yes">
 <vertex x="0" y="0"/>
@@
 <vertex x="59" y="0"/>
 </polygon>
+<wire x1="45.51" y1="50.12" x2="46.802" y2="58.26" width="0" layer="19" extent="1-1"/>
+<wire x1="53.13" y1="50.12" x2="45.51" y2="50.12" width="0" layer="19" extent="1-1"/>
+<wire x1="37.89" y1="50.12" x2="45.51" y2="50.12" width="0" layer="19" extent="1-1"/>
+<wire x1="29.31" y1="50.22" x2="37.89" y2="50.12" width="0" layer="19" extent="1-1"/>
+<wire x1="24.37" y1="45.14" x2="29.31" y2="50.22" width="0" layer="19" extent="1-1"/>
+<wire x1="21.69" y1="50.22" x2="24.37" y2="45.14" width="0" layer="19" extent="1-1"/>
+<wire x1="14.07" y1="50.22" x2="21.69" y2="50.22" width="0" layer="19" extent="1-1"/>
+<wire x1="31.04" y1="59.1" x2="29.31" y2="50.22" width="0" layer="19" extent="1-1"/>
+<wire x1="16.802" y1="58.94" x2="14.07" y2="50.22" width="0" layer="19" extent="1-1"/>
+<wire x1="5.1" y1="57.31" x2="14.07" y2="50.22" width="0" layer="19" extent="1-1"/>
+<wire x1="17.78" y1="30.48" x2="24.37" y2="45.14" width="0" layer="19" extent="1-1"/>
+<wire x1="17.59" y1="19.02" x2="17.78" y2="30.48" width="0" layer="19" extent="1-1"/>
+<wire x1="43.26" y1="30.02" x2="45.51" y2="50.12" width="0" layer="19" extent="1-1"/>
+<wire x1="49.67" y1="25.12" x2="43.26" y2="30.02" width="0" layer="19" extent="1-1"/>
+<wire x1="52.96" y1="18.32" x2="49.67" y2="25.12" width="0" layer="19" extent="1-1"/>
+<wire x1="52.96" y1="10.43" x2="52.96" y2="18.32" width="0" layer="19" extent="1-1"/>
 </signal>
 <signal name="N$2">
@@
 <contactref element="X2" pad="9"/>
 <contactref element="C4" pad="-"/>
-<contactref element="MIDI_PIN_TX-2" pad="1"/>
 <polygon width="0.4064" layer="16" isolate="0.8128">
 <vertex x="0" y="65.66"/>
@@
 <vertex x="58.12" y="65.66"/>
 </polygon>
+<wire x1="50.59" y1="50.12" x2="50.358" y2="58.26" width="0" layer="19" extent="1-1"/>
+<wire x1="42.97" y1="50.12" x2="50.59" y2="50.12" width="0" layer="19" extent="1-1"/>
+<wire x1="35.35" y1="50.12" x2="42.97" y2="50.12" width="0" layer="19" extent="1-1"/>
+<wire x1="26.77" y1="50.22" x2="35.35" y2="50.12" width="0" layer="19" extent="1-1"/>
+<wire x1="19.15" y1="50.22" x2="26.77" y2="50.22" width="0" layer="19" extent="1-1"/>
+<wire x1="11.53" y1="50.22" x2="19.15" y2="50.22" width="0" layer="19" extent="1-1"/>
+<wire x1="5.1" y1="50.53" x2="11.53" y2="50.22" width="0" layer="19" extent="1-1"/>
+<wire x1="54.63" y1="42.5" x2="50.59" y2="50.12" width="0" layer="19" extent="1-1"/>
+<wire x1="5.08" y1="41.91" x2="5.1" y2="50.53" width="0" layer="19" extent="1-1"/>
+<wire x1="20.358" y1="58.94" x2="19.15" y2="50.22" width="0" layer="19" extent="1-1"/>
+<wire x1="36.12" y1="59.1" x2="35.35" y2="50.12" width="0" layer="19" extent="1-1"/>
+<wire x1="28.79" y1="40.29" x2="26.77" y2="50.22" width="0" layer="19" extent="1-1"/>
+<wire x1="17.78" y1="38.1" x2="28.79" y2="40.29" width="0" layer="19" extent="1-1"/>
+<wire x1="35.64" y1="30.02" x2="28.79" y2="40.29" width="0" layer="19" extent="1-1"/>
+<wire x1="17.78" y1="22.86" x2="17.78" y2="38.1" width="0" layer="19" extent="1-1"/>
+<wire x1="54.29" y1="26.5" x2="54.63" y2="42.5" width="0" layer="19" extent="1-1"/>
+<wire x1="49.67" y1="20.04" x2="54.29" y2="26.5" width="0" layer="19" extent="1-1"/>
+<wire x1="18.48" y1="4.7" x2="17.78" y2="22.86" width="0" layer="19" extent="1-1"/>
 </signal>
 <signal name="N$1">
@@
 <wire x1="55.5" y1="10.43" x2="55.5" y2="18.32" width="0.5" layer="1"/>
 </signal>
-<signal name="TX_PIN">
-<contactref element="PIC16F628A" pad="8"/>
-<contactref element="R8" pad="2"/>
-<wire x1="33.5" y1="17" x2="31" y2="14.5" width="0.5" layer="1"/>
-<wire x1="33.5" y1="20" x2="33.5" y2="17" width="0.5" layer="1"/>
-<wire x1="35.5" y1="22" x2="33.5" y2="20" width="0.5" layer="1"/>
-<wire x1="31" y1="14.5" x2="30.83" y2="14.4" width="0.5" layer="1"/>
-<wire x1="35.5" y1="22" x2="35.64" y2="22.4" width="0.5" layer="1"/>
-</signal>
-<signal name="N$11">
-<contactref element="MIDI_PIN_TX-5" pad="1"/>
-<contactref element="R8" pad="1"/>
-<wire x1="13.5" y1="14.5" x2="18" y2="14.5" width="0.5" layer="1"/>
-<wire x1="18" y1="14.5" x2="18.13" y2="14.4" width="0.5" layer="1"/>
-<wire x1="13.5" y1="14.5" x2="13.13" y2="14.32" width="0.5" layer="1"/>
-</signal>
-<signal name="N$12">
-<contactref element="MIDI_PIN_TX-4" pad="1"/>
-<contactref element="R9" pad="1"/>
-<wire x1="13.5" y1="6" x2="17.5" y2="10" width="0.5" layer="1"/>
-<wire x1="17.5" y1="10" x2="17.83" y2="10.16" width="0.5" layer="1"/>
-<wire x1="13.5" y1="6" x2="13.02" y2="5.78" width="0.5" layer="1"/>
-</signal>
 <signal name="N$6">
