File: MIDIServoControllerCircuit/ServoControllerCircuit.brd (EAGLE design)
At the start: 58.8 x 65.7 mm, 26 parts, among them Q1 20MHz, T1 2N3904, X1 SIGNAL-PWR-GND, X2 SIGNAL-PWR-GND

Commit message: Renamed directory to better reflect what files represent
Parts:
- D1: value 1N4198 -> 1N4148
Changed lines of the file:
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@@
 <attribute name="NAME" x="39.279" y="58.8432" size="1.27" layer="25" ratio="10"/>
 </element>
-<element name="D1" library="diode" package="DO35-10" value="1N4198" x="5.08" y="27.94" smashed="yes" rot="R270">
+<element name="D1" library="diode" package="DO35-10" value="1N4148" x="5.08" y="27.94" smashed="yes" rot="R270">
 <attribute name="NAME" x="6.35" y="30.099" size="1.27" layer="25" ratio="10" rot="R270"/>
 </element>
@@
 <vertex x="59" y="0"/>
 </polygon>
-<wire x1="45.51" y1="50.12" x2="46.802" y2="58.26" width="0" layer="19" extent="1-1"/>
-<wire x1="53.13" y1="50.12" x2="45.51" y2="50.12" width="0" layer="19" extent="1-1"/>
-<wire x1="37.89" y1="50.12" x2="45.51" y2="50.12" width="0" layer="19" extent="1-1"/>
-<wire x1="29.31" y1="50.22" x2="37.89" y2="50.12" width="0" layer="19" extent="1-1"/>
-<wire x1="24.37" y1="45.14" x2="29.31" y2="50.22" width="0" layer="19" extent="1-1"/>
-<wire x1="21.69" y1="50.22" x2="24.37" y2="45.14" width="0" layer="19" extent="1-1"/>
-<wire x1="14.07" y1="50.22" x2="21.69" y2="50.22" width="0" layer="19" extent="1-1"/>
-<wire x1="31.04" y1="59.1" x2="29.31" y2="50.22" width="0" layer="19" extent="1-1"/>
-<wire x1="16.802" y1="58.94" x2="14.07" y2="50.22" width="0" layer="19" extent="1-1"/>
-<wire x1="5.1" y1="57.31" x2="14.07" y2="50.22" width="0" layer="19" extent="1-1"/>
-<wire x1="17.78" y1="30.48" x2="24.37" y2="45.14" width="0" layer="19" extent="1-1"/>
-<wire x1="17.59" y1="19.02" x2="17.78" y2="30.48" width="0" layer="19" extent="1-1"/>
-<wire x1="43.26" y1="30.02" x2="45.51" y2="50.12" width="0" layer="19" extent="1-1"/>
-<wire x1="49.67" y1="25.12" x2="43.26" y2="30.02" width="0" layer="19" extent="1-1"/>
-<wire x1="52.96" y1="18.32" x2="49.67" y2="25.12" width="0" layer="19" extent="1-1"/>
-<wire x1="52.96" y1="10.43" x2="52.96" y2="18.32" width="0" layer="19" extent="1-1"/>
 </signal>
 <signal name="N$2">
@@
 <vertex x="58.12" y="65.66"/>
 </polygon>
-<wire x1="50.59" y1="50.12" x2="50.358" y2="58.26" width="0" layer="19" extent="1-1"/>
-<wire x1="42.97" y1="50.12" x2="50.59" y2="50.12" width="0" layer="19" extent="1-1"/>
-<wire x1="35.35" y1="50.12" x2="42.97" y2="50.12" width="0" layer="19" extent="1-1"/>
-<wire x1="26.77" y1="50.22" x2="35.35" y2="50.12" width="0" layer="19" extent="1-1"/>
-<wire x1="19.15" y1="50.22" x2="26.77" y2="50.22" width="0" layer="19" extent="1-1"/>
-<wire x1="11.53" y1="50.22" x2="19.15" y2="50.22" width="0" layer="19" extent="1-1"/>
-<wire x1="5.1" y1="50.53" x2="11.53" y2="50.22" width="0" layer="19" extent="1-1"/>
-<wire x1="54.63" y1="42.5" x2="50.59" y2="50.12" width="0" layer="19" extent="1-1"/>
-<wire x1="5.08" y1="41.91" x2="5.1" y2="50.53" width="0" layer="19" extent="1-1"/>
-<wire x1="20.358" y1="58.94" x2="19.15" y2="50.22" width="0" layer="19" extent="1-1"/>
-<wire x1="36.12" y1="59.1" x2="35.35" y2="50.12" width="0" layer="19" extent="1-1"/>
-<wire x1="28.79" y1="40.29" x2="26.77" y2="50.22" width="0" layer="19" extent="1-1"/>
-<wire x1="17.78" y1="38.1" x2="28.79" y2="40.29" width="0" layer="19" extent="1-1"/>
-<wire x1="35.64" y1="30.02" x2="28.79" y2="40.29" width="0" layer="19" extent="1-1"/>
-<wire x1="17.78" y1="22.86" x2="17.78" y2="38.1" width="0" layer="19" extent="1-1"/>
-<wire x1="54.29" y1="26.5" x2="54.63" y2="42.5" width="0" layer="19" extent="1-1"/>
-<wire x1="49.67" y1="20.04" x2="54.29" y2="26.5" width="0" layer="19" extent="1-1"/>
-<wire x1="18.48" y1="4.7" x2="17.78" y2="22.86" width="0" layer="19" extent="1-1"/>
 </signal>
 <signal name="N$1">

Commit message: Renamed PWM outputs to better match what they go to
Connections:
- net SERVO1 renamed EYEBROW
- net SERVO2 renamed LEFT_LIP_CORNER
- net SERVO3 renamed RIGHT_LIP_CORNER
- net SERVO4 renamed LOWER_JAR
- net SERVO5 renamed EYELIDS
- net SERVO6 renamed UNUSED
Changed lines of the file:
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@@
 <wire x1="49" y1="31.5" x2="49.34" y2="31.29" width="0.5" layer="1"/>
 </signal>
-<signal name="SERVO3">
+<signal name="RIGHT_LIP_CORNER">
 <contactref element="PIC16F628A" pad="1"/>
 <contactref element="X2" pad="7"/>
@@
 <wire x1="40" y1="50" x2="40.43" y2="50.12" width="0.5" layer="1"/>
 </signal>
-<signal name="SERVO1">
+<signal name="EYEBROW">
 <contactref element="PIC16F628A" pad="17"/>
 <contactref element="X2" pad="1"/>
@@
 <wire x1="55.5" y1="50" x2="55.67" y2="50.12" width="0.5" layer="16"/>
 </signal>
-<signal name="SERVO2">
+<signal name="LEFT_LIP_CORNER">
 <contactref element="PIC16F628A" pad="18"/>
 <contactref element="X2" pad="4"/>
@@
 <wire x1="48" y1="50" x2="48.05" y2="50.12" width="0.5" layer="1"/>
 </signal>
-<signal name="SERVO4">
+<signal name="LOWER_JAR">
 <contactref element="PIC16F628A" pad="2"/>
 <contactref element="X1" pad="1"/>
@@
 <wire x1="32" y1="50" x2="31.85" y2="50.22" width="0.5" layer="1"/>
 </signal>
-<signal name="SERVO5">
+<signal name="EYELIDS">
 <contactref element="PIC16F628A" pad="6"/>
 <contactref element="X1" pad="4"/>
@@
 <wire x1="24.5" y1="50" x2="24.23" y2="50.22" width="0.5" layer="1"/>
 </signal>
-<signal name="SERVO6">
+<signal name="UNUSED">
 <contactref element="PIC16F628A" pad="9"/>
 <contactref element="X1" pad="7"/>
